Commit message: Aded my own robot

File: urdf/udacity_bot.xacro (robot description, xacro)
@@ -35,5 +35,5 @@
   </gazebo>
   <joint type="continuous" name="right_wheel_hinge">
-    <origin xyz="0 -0.15 0" rpy="0 0 0"/>
+    <origin xyz="0 -0.5 0" rpy="0 0 0"/>
     <child link="right_wheel"/>
     <parent link="chassis"/>
@@ -66,5 +66,5 @@
   </link>
   <joint type="continuous" name="left_wheel_hinge">
-    <origin xyz="0 0.15 0" rpy="0 0 0"/>
+    <origin xyz="0 0.5 0" rpy="0 0 0"/>
     <child link="left_wheel"/>
     <parent link="chassis"/>
@@ -99,5 +99,5 @@
       <origin xyz="0 0 0" rpy=" 0 0 0"/>
       <geometry>
-        <box size=".4 .2 .1"/>
+        <box size=".4 0.9 .1"/>
       </geometry>
     </visual>
@@ -186,5 +186,5 @@
     </inertial>
     <visual name='visual_hokuyo'>
-      <origin xyz="0.0 0 0" rpy="0 0 0"/>
+      <origin xyz="0.0 0.4 0" rpy="0 0 0"/>
       <geometry>
         <mesh filename="package://udacity_bot/meshes/hokuyo.dae"/>
